Commit message: Переписал контроллер под unitree a1 без редактирования urdf. по-честному. Привел в соответствие прямую и обратную связь

File: src/a1_description/urdf/a1.urdf (robot description, URDF)
Before this commit: robot a1_description, 23 links, 22 joints
Joints:
- joint FL_calf_joint: limit lower=-2.69653369433 upper=-0.916297857297 effort=33.5 velocity=21 -> lower=-2.6965336943312392 upper=-0.9162978572970231 effort=33.5 velocity=21
- joint FL_hip_joint: limit lower=-0.802851455917 upper=0.802851455917 effort=33.5 velocity=21 -> lower=-0.8028514559173915 upper=0.8028514559173915 effort=33.5 velocity=21
- joint FL_thigh_joint: limit lower=-1.0471975512 upper=4.18879020479 effort=33.5 velocity=21 -> lower=-1.0471975511965976 upper=4.1887902047863905 effort=33.5 velocity=21
- joint FR_calf_joint: limit lower=-2.69653369433 upper=-0.916297857297 effort=33.5 velocity=21 -> lower=-2.6965336943312392 upper=-0.9162978572970231 effort=33.5 velocity=21
- joint FR_hip_joint: limit lower=-0.802851455917 upper=0.802851455917 effort=33.5 velocity=21 -> lower=-0.8028514559173915 upper=0.8028514559173915 effort=33.5 velocity=21
- joint FR_thigh_joint: limit lower=-1.0471975512 upper=4.18879020479 effort=33.5 velocity=21 -> lower=-1.0471975511965976 upper=4.1887902047863905 effort=33.5 velocity=21
- joint RL_calf_joint: limit lower=-2.69653369433 upper=-0.916297857297 effort=33.5 velocity=21 -> lower=-2.6965336943312392 upper=-0.9162978572970231 effort=33.5 velocity=21
- joint RL_hip_joint: limit lower=-0.802851455917 upper=0.802851455917 effort=33.5 velocity=21 -> lower=-0.8028514559173915 upper=0.8028514559173915 effort=33.5 velocity=21
- joint RL_thigh_joint: limit lower=-1.0471975512 upper=4.18879020479 effort=33.5 velocity=21 -> lower=-1.0471975511965976 upper=4.1887902047863905 effort=33.5 velocity=21
- joint RR_calf_joint: limit lower=-2.69653369433 upper=-0.916297857297 effort=33.5 velocity=21 -> lower=-2.6965336943312392 upper=-0.9162978572970231 effort=33.5 velocity=21
- joint RR_hip_joint: limit lower=-0.802851455917 upper=0.802851455917 effort=33.5 velocity=21 -> lower=-0.8028514559173915 upper=0.8028514559173915 effort=33.5 velocity=21
- joint RR_thigh_joint: limit lower=-1.0471975512 upper=4.18879020479 effort=33.5 velocity=21 -> lower=-1.0471975511965976 upper=4.1887902047863905 effort=33.5 velocity=21

File: src/a1_description/xacro/const.xacro (robot description, xacro)
@@ -39,5 +39,5 @@
     <xacro:property name="thigh_velocity_max" value="21"/>
     <xacro:property name="thigh_torque_max" value="33.5"/>
-    <xacro:property name="calf_max" value="154.5"/>
+    <xacro:property name="calf_max" value="-52.5"/>
     <xacro:property name="calf_min" value="-154.5"/>
     <xacro:property name="calf_velocity_max" value="21"/>

File: src/a1_description/xacro/leg.xacro (robot description, xacro)
@@ -33,5 +33,5 @@
                     <mesh filename="package://a1_description/meshes/hip.dae" scale="1 1 1"/>
                 </geometry>
-                <!-- <material name="orange"/> -->
+<!--                <material name="orange"/>-->
             </visual>
             <collision>
@@ -68,5 +68,5 @@
             <parent link="${name}_hip"/>
             <child link="${name}_thigh"/>
-            <axis xyz="0 -1 0"/>
+            <axis xyz="0 1 0"/>
             <dynamics damping="${damping}" friction="${friction}"/>
             <limit effort="${thigh_torque_max}" velocity="${thigh_velocity_max}" lower="${thigh_min*PI/180.0}" upper="${thigh_max*PI/180.0}"/>
@@ -83,5 +83,5 @@
                     </xacro:if>
                 </geometry>
-                <!-- <material name="orange"/> -->
+<!--                <material name="orange"/>-->
             </visual>
             <collision>
@@ -104,5 +104,5 @@
             <parent link="${name}_thigh"/>
             <child link="${name}_calf"/>
-            <axis xyz="0 -1 0"/>
+            <axis xyz="0 1 0"/>
             <dynamics damping="${damping}" friction="${friction}"/>
             <limit effort="${calf_torque_max}" velocity="${calf_velocity_max}" lower="${calf_min*PI/180.0}" upper="${calf_max*PI/180.0}"/>
@@ -114,5 +114,5 @@
                     <mesh filename="package://a1_description/meshes/calf.dae" scale="1 1 1"/>
                 </geometry>
-                <!-- <material name="orange"/> -->
+<!--                <material name="orange"/>-->
             </visual>
             <collision>
@@ -142,5 +142,5 @@
                     <sphere radius="${foot_radius-0.01}"/>
                 </geometry>
-                <!-- <material name="orange"/> -->
+<!--                <material name="orange"/>-->
             </visual>
             <collision>

File: src/a1_description/xacro/robot.xacro (robot description, xacro)
@@ -38,5 +38,5 @@
                 <mesh filename="package://a1_description/meshes/trunk.dae" scale="1 1 1"/>
             </geometry>
-            <!-- <material name="orange"/> -->
+<!--            <material name="orange"/>-->
         </visual>
         <collision>

Commit message: Стянуты файлы MIT от Макса, Добавлен пакет unitree msg. Обновлены сабрепы

File: src/a1_description/urdf/a1.urdf (robot description, URDF)
Before this commit: robot a1_description, 23 links, 22 joints
Links:
- added link depth_link; visual mesh filename=package://a1_description/meshes/d435.dae scale=1 1 1
Joints:
- added joint depth_joint: type fixed, parent trunk, child depth_link, origin xyz=0.267 0 0 rpy=2.356194490192345 0 1.5707963267948966

File: src/a1_description/xacro/robot.xacro (robot description, xacro)
@@ -54,4 +54,17 @@
                 izz="${trunk_izz}"/>
         </inertial>
+    </link>
+    <joint name="depth_joint" type="fixed">
+        <origin rpy="${3*PI/4} 0 ${PI/2}" xyz="${trunk_length} 0 0"/>
+        <parent link="trunk"/>
+        <child link="depth_link"/>
+    </joint>
+    <link name="depth_link">
+        <visual>
+            <origin rpy="0 0 0" xyz="0 0 0"/>
+            <geometry>
+                <mesh filename="package://a1_description/meshes/d435.dae" scale="1 1 1"/>
+            </geometry>
+        </visual>
     </link>
     <xacro:if value="${(rolloverProtection == 'true')}">

Commit message: Добавил сенсор глубины

File: src/a1_description/urdf/a1.urdf (robot description, URDF)
Before this commit: robot a1_description, 24 links, 23 joints
Joints:
- joint depth_joint: origin xyz=0.267 0 0 rpy=2.356194490192345 0 1.5707963267948966 -> xyz=0.267 0 0 rpy=0 0.6283185307179586 0

File: src/a1_description/xacro/robot.xacro (robot description, xacro)
@@ -56,5 +56,5 @@
     </link>
     <joint name="depth_joint" type="fixed">
-        <origin rpy="${3*PI/4} 0 ${PI/2}" xyz="${trunk_length} 0 0"/>
+        <origin rpy="0 ${PI/5} 0" xyz="${trunk_length} 0 0"/>
         <parent link="trunk"/>
         <child link="depth_link"/>
@@ -62,5 +62,5 @@
     <link name="depth_link">
         <visual>
-            <origin rpy="0 0 0" xyz="0 0 0"/>
+            <origin rpy="${3*PI/4} 0 ${PI/2}" xyz="0 0 0"/>
             <geometry>
                 <mesh filename="package://a1_description/meshes/d435.dae" scale="1 1 1"/>

Commit message: Обновил сабрепы

File: src/a1_description/urdf/a1.urdf (robot description, URDF)
Before this commit: robot a1_description, 24 links, 23 joints
Joints:
- joint depth_joint: origin xyz=0.267 0 0 rpy=0 0.6283185307179586 0 -> xyz=0.267 0 0 rpy=0 1.5707963267948966 0

File: src/a1_description/xacro/robot.xacro (robot description, xacro)
@@ -56,5 +56,5 @@
     </link>
     <joint name="depth_joint" type="fixed">
-        <origin rpy="0 ${PI/5} 0" xyz="${trunk_length} 0 0"/>
+        <origin rpy="0 ${PI/2} 0" xyz="${trunk_length} 0 0"/>
         <parent link="trunk"/>
         <child link="depth_link"/>
